File: KiCAD/projects/photodiode TIA circuit/photodiode_tia_circuit/photodiode_tia_circuit.kicad_sch (KiCad schematic)
At the start: 3 parts, among them P1 TO46_3PIN, U1 MCP6292, U2 MCP6292

Commit message: changes
Parts:
- added Cdec1: 100nF, Capacitor_THT:C_Disc_D10.5mm_W5.0mm_P5.00mm, symbol Device:C
- added Cf1: DNP, Capacitor_THT:C_Disc_D10.5mm_W5.0mm_P5.00mm, symbol Device:C
- added J_OUT1, J_PWR1: Conn_01x02_Socket, Connector_Molex:Molex_KK-254_AE-6410-02A_1x02_P2.54mm_Vertical, symbol Connector:Conn_01x02_Socket
- added Rf1: 10M R, Resistor_THT:R_Axial_DIN0207_L6.3mm_D2.5mm_P10.16mm_Horizontal, symbol Device:R
- U1: footprint (none) -> Package_DIP:DIP-8_W7.62mm_LongPads
Connections:
- net +3.3V: now also Cdec1.1, J_PWR1.1 (Pin_1)
- net GND: now also P1.2 (GND), Cdec1.2, J_OUT1.2 (Pin_2), J_PWR1.2 (Pin_2)
- net at P1.1 (Cathode), U1.2 (-): now also Cf1.1, Rf1.2
- net at U1.1: now also Cf1.2, J_OUT1.1 (Pin_1), Rf1.1
Other:
- moved on the sheet: P1, U1A

Commit message: manufacture documents and 3d model step file
Parts:
- added Rf2: 100k, Resistor_THT:R_Axial_DIN0207_L6.3mm_D2.5mm_P10.16mm_Horizontal, symbol Device:R
- added Rf3: 1.8k, Resistor_THT:R_Axial_DIN0207_L6.3mm_D2.5mm_P10.16mm_Horizontal, symbol Device:R
- Cdec1: value 100nF -> 0.1uF
- Cf1: value DNP -> 2pF
- Rf1: value 10M R -> 470k
- U1: renamed from U2; footprint (none) -> Package_DIP:DIP-8_W7.62mm_LongPads
Connections:
- net GND: now also Rf3.2; no longer U1.5 (+), U1.6 (-), U1.7
- net at Cf1.2, Rf1.1, U1.1: now also U1.5 (+); no longer J_OUT1.1 (Pin_1)
- new net: J_OUT1.1 (Pin_1), Rf2.1, U1.7
- new net: Rf2.2, Rf3.1, U1.6 (-)
Other:
- moved on the sheet: J_OUT1, U1B
