File: KiCAD/projects/photodiode TIA circuit/photodiode_tia_circuit/photodiode_tia_circuit.kicad_sch (KiCad schematic)
At the start: 9 parts, among them J1 Conn_01x05_Socket, J2 Conn_01x03_Socket, P1 TO46_3PIN, U1 MCP6292

Commit message: latest version
Parts:
- added Cdec2, Cdec5: 10uF, Capacitor_THT:C_Disc_D10.5mm_W5.0mm_P5.00mm, symbol Device:C
- added Cdec3, Cdec4: 100nF, Capacitor_THT:C_Disc_D10.5mm_W5.0mm_P5.00mm, symbol Device:C
- added Rf4: 5.6k, Resistor_THT:R_Axial_DIN0207_L6.3mm_D2.5mm_P10.16mm_Horizontal, symbol Device:R
- added Rf5: 1k, Resistor_THT:R_Axial_DIN0207_L6.3mm_D2.5mm_P10.16mm_Horizontal, symbol Device:R
- Cdec1: value 0.1uF -> 100nF
Connections:
- net +3.3V: now also Cdec2.2, Cdec3.2, Rf4.1
- net GND: now also Cdec2.1, Cdec3.1, Cdec4.1, Cdec5.1, Rf5.2; no longer Rf3.2, U1.3 (+)
- new net: Cdec4.2, Cdec5.2, Rf3.2, Rf4.2, Rf5.1, U1.3 (+)
