File: KiCAD/projects/photodiode TIA circuit/photodiode_tia_circuit/photodiode_tia_circuit_v2.kicad_sch (KiCad schematic)
At the start: 9 parts, among them J1 Conn_01x05_Socket, J2 Conn_01x03_Socket, P1 TO46_3PIN, U1 MCP6292

Commit message: new
Parts:
- removed J1: Conn_01x05_Socket, Connector_JST:JST_EH_S5B-EH_1x05_P2.50mm_Horizontal, symbol Connector:Conn_01x05_Socket
- removed J2: Conn_01x03_Socket, Connector_JST:JST_EH_S3B-EH_1x03_P2.50mm_Horizontal, symbol Connector:Conn_01x03_Socket
- added J_OUT1, J_PWR1: Conn_01x02_Socket, Connector_Molex:Molex_KK-254_AE-6410-02A_1x02_P2.54mm_Vertical, symbol Connector:Conn_01x02_Socket
Connections:
- net +3.3V: now also J_PWR1.1 (Pin_1)
- net GND: now also J_OUT1.2 (Pin_2), J_PWR1.2 (Pin_2)
- net at Rf2.1, U1.7: now also J_OUT1.1 (Pin_1)
