File: KiCAD/projects/photodiode TIA circuit/photodiode_tia_circuit/photodiode_tia_circuit_simulation.kicad_sch (KiCad schematic)
At the start: 10 parts, among them U2 ${SIM.PARAMS}, U3 ${SIM.PARAMS}

Commit message: latest version
Parts:
- removed V3: 1.65, symbol Simulation_SPICE:VDC
- added Cf3: 10uF, Capacitor_THT:C_Disc_D10.5mm_W5.0mm_P5.00mm, symbol Device:C
- added Rf2: 5.6k, Resistor_THT:R_Axial_DIN0207_L6.3mm_D2.5mm_P10.16mm_Horizontal, symbol Device:R
- added Rf5: 50k, Resistor_THT:R_Axial_DIN0207_L6.3mm_D2.5mm_P10.16mm_Horizontal, symbol Device:R
- Cf2: value 2pF -> 100nF
- Rf4: value 100 -> 1k
Connections:
- net 3V3: now also Rf2.1
- net GND: now also Cf3.1; no longer U2.1 (+)
- net pulse_current: no longer Cf2.2, Rf4.1
- net stage_2_output: now also Rf5.1
- net at Rf3.1, U3.2 (-): now also Rf5.2
- net at Rf3.2: now also Cf2.2, Rf4.1, U2.1 (+), Cf3.2, Rf2.2
Other:
- note added: ".param period=990us .param width=10u .param amp=200n .param r0=1m .param dr=1m"
- note removed: ".param period=100us .param width=10u .param amp=200n .param r0=1m .param dr=0.05m"
