File: KiCAD/projects/photodiode TIA circuit/photodiode_tia_circuit/photodiode_tia_circuit_v3.kicad_sch (KiCad schematic)
At the start: 15 parts, among them J1 Conn_01x05_Socket, J2 Conn_01x03_Socket, P1 TO46_3PIN, U1 OPA2320

Commit message: latest TIA
Parts:
- Cdec1, Cdec3, Cdec4, Cf1: footprint Capacitor_THT:C_Disc_D5.0mm_W2.5mm_P2.50mm -> Capacitor_THT:C_Disc_D10.5mm_W5.0mm_P5.00mm
- Rf2: value 180k -> 100k
- U1: value OPA2320 -> MCP6292; footprint OPA2320:D8-M -> Package_DIP:DIP-8_W7.62mm_LongPads
Connections:
- net GND: now also P1.2 (GND), P1.3 (Anode)
- net at Cdec4.2, Cdec5.2, Rf3.2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: no longer P1.2 (GND), P1.3 (Anode)
Changed lines of the file:
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@@
-	)
-	(junction
-		(at 102.87 156.21)
-		(diameter 0)
-		(color 0 0 0 0)
 	)
 	(junction
@@
 		(color 0 0 0 0)
 	)
-	(junction
-		(at 113.03 156.21)
-		(diameter 0)
-		(color 0 0 0 0)
-	)
 	(wire
 		(pts
@@
 	(wire
 		(pts
-			(xy 96.52 156.21) (xy 102.87 156.21)
+			(xy 96.52 156.21) (xy 116.84 156.21)
 		)
 		(stroke
@@
 	(wire
 		(pts
-			(xy 113.03 156.21) (xy 116.84 156.21)
-		)
-		(stroke
-			(width 0)
-			(type default)
-		)
-	)
-	(wire
-		(pts
 			(xy 87.63 156.21) (xy 96.52 156.21)
 		)
@@
 	(wire
 		(pts
-			(xy 102.87 156.21) (xy 113.03 156.21)
+			(xy 102.87 133.35) (xy 102.87 137.16)
 		)
 		(stroke
@@
 	(wire
 		(pts
-			(xy 113.03 127) (xy 113.03 156.21)
-		)
-		(stroke
-			(width 0)
-			(type default)
-		)
-	)
-	(wire
-		(pts
 			(xy 118.11 62.23) (xy 118.11 69.85)
 		)
@@
 	(wire
 		(pts
-			(xy 102.87 133.35) (xy 102.87 156.21)
-		)
-		(stroke
-			(width 0)
-			(type default)
-		)
-	)
-	(wire
-		(pts
 			(xy 114.3 91.44) (xy 114.3 102.87)
 		)
@@
 		(pts
 			(xy 102.87 114.3) (xy 102.87 120.65)
+		)
+		(stroke
+			(width 0)
+			(type default)
+		)
+	)
+	(wire
+		(pts
+			(xy 113.03 127) (xy 113.03 128.27)
 		)
 		(stroke
@@
 			)
 		)
-		(property "Value" "OPA2320"
+		(property "Value" "MCP6292"
 			(at 104.14 67.3099 0)
 			(show_name no)
@@
 			)
 		)
-		(property "Footprint" "OPA2320:D8-M"
+		(property "Footprint" "Package_DIP:DIP-8_W7.62mm_LongPads"
 			(at 105.41 66.04 0)
 			(hide yes)
@@
 			)
 		)
-		(property "Footprint" "Capacitor_THT:C_Disc_D5.0mm_W2.5mm_P2.50mm"
+		(property "Footprint" "Capacitor_THT:C_Disc_D10.5mm_W5.0mm_P5.00mm"
 			(at 127 90.4748 0)
 			(hide yes)
@@
 			)
 		)
-		(property "Value" "OPA2320"
+		(property "Value" "MCP6292"
 			(at 151.13 111.76 0)
 			(show_name no)
@@
 			)
 		)
-		(property "Footprint" "OPA2320:D8-M"
+		(property "Footprint" "Package_DIP:DIP-8_W7.62mm_LongPads"
 			(at 151.13 119.38 0)
 			(hide yes)
@@
 			)
 		)
-		(property "Footprint" "Capacitor_THT:C_Disc_D5.0mm_W2.5mm_P2.50mm"
+		(property "Footprint" "Capacitor_THT:C_Disc_D10.5mm_W5.0mm_P5.00mm"
 			(at 86.6648 156.21 0)
 			(hide yes)
@@
 	)
 	(symbol
+		(lib_id "power:GND")
+		(at 102.87 137.16 0)
+		(unit 1)
+		(body_style 1)
+		(exclude_from_sim no)
+		(in_bom yes)
+		(on_board yes)
+		(in_pos_files yes)
+		(dnp no)
+		(property "Reference" "#PWR06"
+			(at 102.87 143.51 0)
+			(hide yes)
+			(show_name no)
+			(do_not_autoplace no)
+			(effects
+				(font
+					(size 1.27 1.27)
+				)
+			)
+		)
+		(property "Value" "GND"
+			(at 99.314 139.192 0)
+			(show_name no)
+			(do_not_autoplace no)
+			(effects
+				(font
+					(size 1.27 1.27)
+				)
+			)
+		)
+		(property "Footprint" ""
+			(at 102.87 137.16 0)
+			(hide yes)
+			(show_name no)
+			(do_not_autoplace no)
+			(effects
+				(font
+					(size 1.27 1.27)
+				)
+			)
+		)
+		(property "Datasheet" ""
+			(at 102.87 137.16 0)
+			(hide yes)
+			(show_name no)
+			(do_not_autoplace no)
+			(effects
+				(font
+					(size 1.27 1.27)
+				)
+			)
+		)
+		(property "Description" "Power symbol creates a global label with name \"GND\" , ground"
+			(at 102.87 137.16 0)
+			(hide yes)
+			(show_name no)
+			(do_not_autoplace no)
+			(effects
+				(font
+					(size 1.27 1.27)
+				)
+			)
+		)
+		(pin "1"
+		)
+		(instances
+			(project "photodiode_tia_circuit"
+				(path "/c9490f31-99a0-4a89-8aa1-95c2524c298c"
+					(reference "#PWR06")
+					(unit 1)
+				)
+			)
+		)
+	)
+	(symbol
 		(lib_id "power:+3.3V")
 		(at 73.66 144.78 0)
@@
 			)
 		)
-		(property "Value" "OPA2320"
+		(property "Value" "MCP6292"
 			(at 124.714 123.952 0)
 			(show_name no)
@@
 			)
 		)
-		(property "Footprint" "OPA2320:D8-M"
+		(property "Footprint" "Package_DIP:DIP-8_W7.62mm_LongPads"
 			(at 125.73 116.84 0)
 			(hide yes)
@@
 	)
 	(symbol
+		(lib_id "power:GND")
+		(at 113.03 128.27 0)
+		(unit 1)
+		(body_style 1)
+		(exclude_from_sim no)
+		(in_bom yes)
+		(on_board yes)
+		(in_pos_files yes)
+		(dnp no)
+		(fields_autoplaced yes)
+		(property "Reference" "#PWR09"
+			(at 113.03 134.62 0)
+			(hide yes)
+			(show_name no)
+			(do_not_autoplace no)
+			(effects
+				(font
+					(size 1.27 1.27)
+				)
+			)
+		)
+		(property "Value" "GND"
+			(at 113.03 133.35 0)
+			(show_name no)
+			(do_not_autoplace no)
+			(effects
+				(font
+					(size 1.27 1.27)
+				)
+			)
+		)
+		(property "Footprint" ""
+			(at 113.03 128.27 0)
+			(hide yes)
+			(show_name no)
+			(do_not_autoplace no)
+			(effects
+				(font
+					(size 1.27 1.27)
+				)
+			)
+		)
+		(property "Datasheet" ""
+			(at 113.03 128.27 0)
+			(hide yes)
+			(show_name no)
+			(do_not_autoplace no)
+			(effects
+				(font
+					(size 1.27 1.27)
+				)
+			)
+		)
+		(property "Description" "Power symbol creates a global label with name \"GND\" , ground"
+			(at 113.03 128.27 0)
+			(hide yes)
+			(show_name no)
+			(do_not_autoplace no)
+			(effects
+				(font
+					(size 1.27 1.27)
+				)
+			)
+		)
+		(pin "1"
+		)
+		(instances
+			(project "photodiode_tia_circuit"
+				(path "/c9490f31-99a0-4a89-8aa1-95c2524c298c"
+					(reference "#PWR09")
+					(unit 1)
+				)
+			)
+		)
+	)
+	(symbol
 		(lib_id "power:+3.3V")
 		(at 102.87 58.42 0)
@@
 			)
 		)
-		(property "Footprint" "Capacitor_THT:C_Disc_D5.0mm_W2.5mm_P2.50mm"
+		(property "Footprint" "Capacitor_THT:C_Disc_D10.5mm_W5.0mm_P5.00mm"
 			(at 118.11 61.2648 0)
 			(hide yes)
@@
 			)
 		)
-		(property "Value" "180k"
+		(property "Value" "100k"
 			(at 148.59 130.81 90)
 			(show_name no)
@@
 			)
 		)
-		(property "Footprint" "Capacitor_THT:C_Disc_D5.0mm_W2.5mm_P2.50mm"
+		(property "Footprint" "Capacitor_THT:C_Disc_D10.5mm_W5.0mm_P5.00mm"
 			(at 184.4548 105.41 0)
 			(hide yes)
