File: KiCAD/projects/MYOSA_breakout/MYOSA_breakout.kicad_sch (KiCad schematic)
At the start: 23 parts, among them J1 Conn_01x04_Socket, J2 Conn_01x05_Socket, J3 PSU, Q1 IRLZ44N, SW1 Batt/PSU_switch, SW2 USB/REG_switch, U2 D24V22F5

Commit message: MYOSA skeleton PCB
Parts:
- removed J3: PSU, symbol Connector:Conn_01x02_Socket
- removed SW1: Batt/PSU_switch, symbol Switch:SW_DPDT_x2
- removed SW2: USB/REG_switch, symbol Switch:SW_DPDT_x2
- added J3: PSU_9V, Connector:Banana_Cliff_FCR7350R_S16N-PC_Horizontal, symbol Connector:Conn_01x01_Socket
- added J4: PSU_GND, Connector:Banana_Cliff_FCR7350B_S16N-PC_Horizontal, symbol Connector:Conn_01x01_Socket
- added R5: 200, Resistor_THT:R_Axial_DIN0207_L6.3mm_D2.5mm_P7.62mm_Horizontal, symbol Device:R
- added SW1: Batt/PSU_switch, Button_Switch_THT:SW_Slide_SPDT_Straight_CK_OS102011MS2Q, symbol Switch:SW_SPDT
- added SW2: USB/REG_switch, Button_Switch_THT:SW_Slide_SPDT_Straight_CK_OS102011MS2Q, symbol Switch:SW_SPDT
- added TP6: PhotoIn_TestPoint, TestPoint:TestPoint_Pad_2.0x2.0mm, symbol Connector:TestPoint
- ADC_cap1: renamed from ADC_cap; footprint (none) -> Capacitor_THT:C_Disc_D5.0mm_W2.5mm_P5.00mm
- ADC_pulldown1: renamed from ADC_pulldown; footprint (none) -> Resistor_THT:R_Axial_DIN0207_L6.3mm_D2.5mm_P7.62mm_Horizontal
- C1: value C -> 100nF; footprint (none) -> Capacitor_THT:C_Disc_D5.0mm_W2.5mm_P5.00mm
- C2: footprint (none) -> Capacitor_THT:C_Disc_D5.0mm_W2.5mm_P5.00mm
- R1, R2, R3, R4: footprint (none) -> Resistor_THT:R_Axial_DIN0207_L6.3mm_D2.5mm_P7.62mm_Horizontal
- TP3, TP4: footprint (none) -> TestPoint:TestPoint_Pad_2.0x2.0mm
Connections:
- net 5V: now also SW2.2 (B)
- net GND: now also J4.1 (Pin_1), R5.2; no longer C1.2
- net Photo_IN: now also TP6.1
- net Vin_SRC: now also SW1.2 (B)
- net at BT1.1 (+): now also SW1.3 (C)
- net at U1.2 (VIN): now also SW2.3 (C)
- new net: J3.1 (Pin_1), SW1.1 (A)
- new net: C1.2, R5.1
Other:
- moved on the sheet: J1, J2

Commit message: MYOSA PCB v1
Parts:
- removed TP4: 3V3_TestPoint, TestPoint:TestPoint_Pad_2.0x2.0mm, symbol Connector:TestPoint
- 5V_Reg_LED1: renamed from D1; footprint (none) -> LED_THT:LED_D5.0mm
- CON_BMP180_1: renamed from J1; footprint (none) -> Connector_JST:JST_EH_S4B-EH_1x04_P2.50mm_Horizontal
- CON_LED_Photodiode1: renamed from J2; footprint (none) -> Connector_JST:JST_EH_S5B-EH_1x05_P2.50mm_Horizontal
- TP1, TP3, TP5, TP6: footprint TestPoint:TestPoint_Pad_2.0x2.0mm -> TestPoint:TestPoint_Loop_D2.50mm_Drill1.85mm
- renumbered C2 to C_3V3_out1, ADC_cap1 to C_ADC_cap1, C1 to C_Vin1, ADC_pulldown1 to R_ADC_pulldown1, R2 to R_FET_Gate1, R3 to R_FET_pulldown1, R5 to R_Vin1, R4 to R_reg_LED1, R1 to R_series_MWIR_LED1, SW1 to SW_BAT/PSU1, SW2 to SW_USB1
Changed lines of the file:
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@@
 	)
 	(junction
-		(at 100.33 106.68)
-		(diameter 0)
-		(color 0 0 0 0)
-	)
-	(junction
 		(at 48.26 133.35)
 		(diameter 0)
@@
 	(wire
 		(pts
-			(xy 100.33 106.68) (xy 95.25 106.68)
+			(xy 95.25 106.68) (xy 113.03 106.68)
 		)
 		(stroke
@@
 	(wire
 		(pts
-			(xy 100.33 106.68) (xy 113.03 106.68)
-		)
-		(stroke
-			(width 0)
-			(type default)
-		)
-	)
-	(wire
-		(pts
 			(xy 190.5 101.6) (xy 203.2 101.6)
 		)
@@
 		(dnp no)
 		(fields_autoplaced yes)
-		(property "Reference" "J2"
+		(property "Reference" "CON_LED_Photodiode1"
 			(at 209.55 105.4099 0)
 			(effects
@@
 			)
 		)
-		(property "Footprint" ""
+		(property "Footprint" "Connector_JST:JST_EH_S5B-EH_1x05_P2.50mm_Horizontal"
 			(at 208.28 106.68 0)
 			(effects
@@
 			(project ""
 				(path "/2a0dcf9b-71c0-4203-830a-99306309dd4e"
-					(reference "J2")
+					(reference "CON_LED_Photodiode1")
 					(unit 1)
 				)
@@
 		(dnp no)
 		(fields_autoplaced yes)
-		(property "Reference" "ADC_cap1"
+		(property "Reference" "C_ADC_cap1"
 			(at 162.56 140.9699 0)
 			(effects
@@
 			(project "MYOSA_breakout"
 				(path "/2a0dcf9b-71c0-4203-830a-99306309dd4e"
-					(reference "ADC_cap1")
+					(reference "C_ADC_cap1")
 					(unit 1)
 				)
@@
 		(on_board yes)
 		(dnp no)
-		(property "Reference" "SW1"
+		(property "Reference" "SW_BAT/PSU1"
 			(at 51.562 27.178 0)
 			(effects
@@
 			(project ""
 				(path "/2a0dcf9b-71c0-4203-830a-99306309dd4e"
-					(reference "SW1")
+					(reference "SW_BAT/PSU1")
 					(unit 1)
 				)
@@
 			)
 		)
-		(property "Footprint" "TestPoint:TestPoint_Pad_2.0x2.0mm"
+		(property "Footprint" "TestPoint:TestPoint_Loop_D2.50mm_Drill1.85mm"
 			(at 53.34 133.35 0)
 			(effects
@@
 			)
 		)
-		(property "Footprint" "TestPoint:TestPoint_Pad_2.0x2.0mm"
+		(property "Footprint" "TestPoint:TestPoint_Loop_D2.50mm_Drill1.85mm"
 			(at 160.02 138.43 0)
 			(effects
@@
 		(dnp no)
 		(fields_autoplaced yes)
-		(property "Reference" "C1"
+		(property "Reference" "C_Vin1"
 			(at 60.96 38.0999 0)
 			(effects
@@
 			(project ""
 				(path "/2a0dcf9b-71c0-4203-830a-99306309dd4e"
-					(reference "C1")
+					(reference "C_Vin1")
 					(unit 1)
 				)
@@
 		(dnp no)
 		(fields_autoplaced yes)
-		(property "Reference" "R1"
+		(property "Reference" "R_series_MWIR_LED1"
 			(at 67.31 109.2199 0)
 			(effects
@@
 			(project ""
 				(path "/2a0dcf9b-71c0-4203-830a-99306309dd4e"
-					(reference "R1")
+					(reference "R_series_MWIR_LED1")
 					(unit 1)
 				)
@@
 			)
 		)
-		(property "Footprint" "TestPoint:TestPoint_Pad_2.0x2.0mm"
+		(property "Footprint" "TestPoint:TestPoint_Loop_D2.50mm_Drill1.85mm"
 			(at 92.71 44.45 0)
 			(effects
@@
 			)
 		)
-		(property "Footprint" "TestPoint:TestPoint_Pad_2.0x2.0mm"
+		(property "Footprint" "TestPoint:TestPoint_Loop_D2.50mm_Drill1.85mm"
 			(at 64.77 113.03 0)
 			(effects
@@
 		(dnp no)
 		(fields_autoplaced yes)
-		(property "Reference" "R3"
+		(property "Reference" "R_FET_pulldown1"
 			(at 50.8 143.5099 0)
 			(effects
@@
 			(project ""
 				(path "/2a0dcf9b-71c0-4203-830a-99306309dd4e"
-					(reference "R3")
+					(reference "R_FET_pulldown1")
 					(unit 1)
 				)
@@
 		)
 		(property "Value" "PSU_9V"
-			(at 26.162 44.45 0)
+			(at 25.654 44.196 0)
 			(effects
 				(font
@@
 		(dnp no)
 		(fields_autoplaced yes)
-		(property "Reference" "J1"
+		(property "Reference" "CON_BMP180_1"
 			(at 208.28 128.2699 0)
 			(effects
@@
 			)
 		)
-		(property "Footprint" ""
+		(property "Footprint" "Connector_JST:JST_EH_S4B-EH_1x04_P2.50mm_Horizontal"
 			(at 207.01 128.27 0)
 			(effects
@@
 			(project ""
 				(path "/2a0dcf9b-71c0-4203-830a-99306309dd4e"
-					(reference "J1")
+					(reference "CON_BMP180_1")
 					(unit 1)
 				)
@@
 		(dnp no)
 		(fields_autoplaced yes)
-		(property "Reference" "SW2"
+		(property "Reference" "SW_USB1"
 			(at 149.86 100.33 0)
 			(effects
@@
 			(project ""
 				(path "/2a0dcf9b-71c0-4203-830a-99306309dd4e"
-					(reference "SW2")
-					(unit 1)
-				)
-			)
-		)
-	)
-	(symbol
-		(lib_id "Connector:TestPoint")
-		(at 100.33 106.68 0)
-		(unit 1)
-		(exclude_from_sim no)
-		(in_bom yes)
-		(on_board yes)
-		(dnp no)
-		(property "Reference" "TP4"
-			(at 100.584 100.33 0)
-			(effects
-				(font
-					(size 1.27 1.27)
-				)
-			)
-		)
-		(property "Value" "3V3_TestPoint"
-			(at 100.584 98.298 0)
-			(effects
-				(font
-					(size 1.27 1.27)
-				)
-			)
-		)
-		(property "Footprint" "TestPoint:TestPoint_Pad_2.0x2.0mm"
-			(at 105.41 106.68 0)
-			(effects
-				(font
-					(size 1.27 1.27)
-				)
-				(hide yes)
-			)
-		)
-		(property "Datasheet" "~"
-			(at 105.41 106.68 0)
-			(effects
-				(font
-					(size 1.27 1.27)
-				)
-				(hide yes)
-			)
-		)
-		(property "Description" "test point"
-			(at 100.33 106.68 0)
-			(effects
-				(font
-					(size 1.27 1.27)
-				)
-				(hide yes)
-			)
-		)
-		(pin "1"
-		)
-		(instances
-			(project "MYOSA_breakout"
-				(path "/2a0dcf9b-71c0-4203-830a-99306309dd4e"
-					(reference "TP4")
+					(reference "SW_USB1")
 					(unit 1)
 				)
@@
 		(on_board yes)
 		(dnp no)
-		(fields_autoplaced yes)
-		(property "Reference" "C2"
-			(at 99.06 109.2199 0)
+		(property "Reference" "C_3V3_out1"
+			(at 98.044 114.046 0)
 			(effects
 				(font
@@
 		)
 		(property "Value" "C"
-			(at 99.06 111.7599 0)
+			(at 98.298 111.506 0)
 			(effects
 				(font
@@
 			(project "MYOSA_breakout"
 				(path "/2a0dcf9b-71c0-4203-830a-99306309dd4e"
-					(reference "C2")
+					(reference "C_3V3_out1")
 					(unit 1)
 				)
@@
 		(dnp no)
 		(fields_autoplaced yes)
-		(property "Reference" "R4"
+		(property "Reference" "R_reg_LED1"
 			(at 95.25 54.6099 0)
 			(effects
@@
 			(project ""
 				(path "/2a0dcf9b-71c0-4203-830a-99306309dd4e"
-					(reference "R4")
+					(reference "R_reg_LED1")
 					(unit 1)
 				)
@@
 		(dnp no)
 		(fields_autoplaced yes)
-		(property "Reference" "ADC_pulldown1"
+		(property "Reference" "R_ADC_pulldown1"
 			(at 143.51 140.9699 0)
 			(effects
@@
 			(project ""
 				(path "/2a0dcf9b-71c0-4203-830a-99306309dd4e"
-					(reference "ADC_pulldown1")
+					(reference "R_ADC_pulldown1")
 					(unit 1)
 				)
@@
 		(dnp no)
 		(fields_autoplaced yes)
-		(property "Reference" "R2"
+		(property "Reference" "R_FET_Gate1"
 			(at 35.56 127 90)
 			(effects
@@
 			(project ""
 				(path "/2a0dcf9b-71c0-4203-830a-99306309dd4e"
-					(reference "R2")
+					(reference "R_FET_Gate1")
 					(unit 1)
 				)
@@
 		(dnp no)
 		(fields_autoplaced yes)
-		(property "Reference" "D1"
+		(property "Reference" "5V_Reg_LED1"
 			(at 96.52 63.8174 90)
 			(effects
@@
 			)
 		)
-		(property "Footprint" ""
+		(property "Footprint" "LED_THT:LED_D5.0mm"
 			(at 92.71 63.5 0)
 			(effects
@@
 			(project ""
 				(path "/2a0dcf9b-71c0-4203-830a-99306309dd4e"
-					(reference "D1")
+					(reference "5V_Reg_LED1")
 					(unit 1)
 				)
@@
 		(dnp no)
 		(fields_autoplaced yes)
-		(property "Reference" "R5"
+		(property "Reference" "R_Vin1"
 			(at 59.69 45.7199 0)
 			(effects
@@
 			(project "MYOSA_breakout"
 				(path "/2a0dcf9b-71c0-4203-830a-99306309dd4e"
-					(reference "R5")
+					(reference "R_Vin1")
 					(unit 1)
 				)

Commit message: KiCAD Updates + Manufacturing
Parts:
- removed CON_BMP180_1: Conn_01x04_Socket, Connector_JST:JST_EH_S4B-EH_1x04_P2.50mm_Horizontal, symbol Connector:Conn_01x04_Socket
- J3: footprint Connector:Banana_Cliff_FCR7350R_S16N-PC_Horizontal -> Connector:Banana_Jack_1Pin
- J4: footprint Connector:Banana_Cliff_FCR7350B_S16N-PC_Horizontal -> Connector:Banana_Jack_1Pin
- SW_BAT/PSU1, SW_USB1: footprint Button_Switch_THT:SW_Slide_SPDT_Straight_CK_OS102011MS2Q -> Button_Switch_THT:SW_Slide-03_Wuerth-WS-SLTV_10x2.5x6.4_P2.54mm
Connections:
- net CLK: no longer names the net of U1.15 (SCL)
- net DAT: no longer names the net of U1.18 (SDA)
- no-connect marks 21 -> 22
Other:
- note removed: "BMP180"
